Commit message: Added admittance control to dmp_ur10_controller

File: c++/as64_ws/src/lib/ur_robot/universal_robot/universal_robot/ur_description/urdf/ur10.urdf.xacro (robot description, xacro)
@@ -291,4 +291,29 @@
       <child link="${prefix}tool0"/>
     </joint>
+    <!-- Joint Force Torque Sensor -->
+    <joint name="${prefix}optoforce_Connection" type="fixed">
+		  <parent link="${prefix}tool0" />
+		  <child link = "${prefix}optoforce_frame" />
+		  <origin xyz="0 0.0 0.015" rpy="0 0 -1.57" />
+    </joint>
+    <link name="${prefix}optoforce_frame">
+      <collision>
+        <origin xyz="0 0 0" rpy="0 0 0"/>
+        <geometry>
+      <cylinder length="0" radius="0"/>
+        </geometry>
+      </collision>
+      <visual>
+        <origin xyz="0 0 0" rpy="0 0 0"/>
+        <geometry>
+      <cylinder length="0.03" radius="0.035"/>
+        </geometry>
+      </visual>
+      <inertial>
+        <mass value="0.1" />
+        <origin xyz="0 0 0" rpy="0 0 0"/>
+        <inertia ixx="1e-6" ixy="0" ixz="0" iyy="1e-6" iyz="0" izz="1e-6" />
+      </inertial>
+</link>
   </xacro:macro>
 </robot>

Commit message: Changed optoforce callibration, fixed a bug in admittance init andadded reject, halt and modify admittance modes in model run

File: c++/as64_ws/src/lib/ur_robot/universal_robot/universal_robot/ur_description/urdf/ur10.urdf.xacro (robot description, xacro)
@@ -295,5 +295,5 @@
 		  <parent link="${prefix}tool0" />
 		  <child link = "${prefix}optoforce_frame" />
-		  <origin xyz="0 0.0 0.015" rpy="0 0 -1.57" />
+		  <origin xyz="0 0.0 0.015" rpy="0 0 0" />
     </joint>
     <link name="${prefix}optoforce_frame">
